File: hw/ver1/rf_controller.kicad_sch (KiCad schematic)
At the start: 1 part, among them U2 ESP32-S2-MINI-1

Commit message: Add virtual environment. Layout some schematic ideas. Add design doc for LTC7871.
Parts:
- U2: footprint Espressif:ESP32-S2-MINI-1_HandSoldering -> PCM_Espressif:ESP32-S2-MINI-1
