File: hw/ver1/PowerStage/mppt_controller.kicad_sch (KiCad schematic)
At the start: 1 part, among them U1 RP2040

Commit message: Split controller from the power stage. Get a better high level system flow.
Parts:
- removed U1: RP2040, Package_DFN_QFN:QFN-56-1EP_7x7mm_P0.4mm_EP3.2x3.2mm, symbol MCU_RaspberryPi:RP2040
Changed lines of the file:
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@@
 	(generator_version "8.0")
 	(paper "A4")
-	(symbol
-		(lib_id "MCU_RaspberryPi:RP2040")
-		(at 146.685 80.645 0)
-		(unit 1)
-		(exclude_from_sim no)
-		(in_bom yes)
-		(on_board yes)
-		(dnp no)
-		(fields_autoplaced yes)
-		(property "Reference" "U1"
-			(at 148.8791 125.095 0)
-			(effects
-				(font
-					(size 1.27 1.27)
-				)
-				(justify left)
-			)
-		)
-		(property "Value" "RP2040"
-			(at 148.8791 127.635 0)
-			(effects
-				(font
-					(size 1.27 1.27)
-				)
-				(justify left)
-			)
-		)
-		(property "Footprint" "Package_DFN_QFN:QFN-56-1EP_7x7mm_P0.4mm_EP3.2x3.2mm"
-			(at 146.685 80.645 0)
-			(effects
-				(font
-					(size 1.27 1.27)
-				)
-				(hide yes)
-			)
-		)
-		(property "Datasheet" "https://datasheets.raspberrypi.com/rp2040/rp2040-datasheet.pdf"
-			(at 146.685 80.645 0)
-			(effects
-				(font
-					(size 1.27 1.27)
-				)
-				(hide yes)
-			)
-		)
-		(property "Description" "A microcontroller by Raspberry Pi"
-			(at 146.685 80.645 0)
-			(effects
-				(font
-					(size 1.27 1.27)
-				)
-				(hide yes)
-			)
-		)
-		(pin "53"
-		)
-		(pin "5"
-		)
-		(pin "55"
-		)
-		(pin "12"
-		)
-		(pin "33"
-		)
-		(pin "41"
-		)
-		(pin "24"
-		)
-		(pin "40"
-		)
-		(pin "46"
-		)
-		(pin "2"
-		)
-		(pin "19"
-		)
-		(pin "48"
-		)
-		(pin "44"
-		)
-		(pin "14"
-		)
-		(pin "23"
-		)
-		(pin "47"
-		)
-		(pin "45"
-		)
-		(pin "50"
-		)
-		(pin "20"
-		)
-		(pin "27"
-		)
-		(pin "49"
-		)
-		(pin "21"
-		)
-		(pin "51"
-		)
-		(pin "54"
-		)
-		(pin "17"
-		)
-		(pin "57"
-		)
-		(pin "6"
-		)
-		(pin "31"
-		)
-		(pin "8"
-		)
-		(pin "43"
-		)
-		(pin "18"
-		)
-		(pin "36"
-		)
-		(pin "32"
-		)
-		(pin "4"
-		)
-		(pin "38"
-		)
-		(pin "52"
-		)
-		(pin "7"
-		)
-		(pin "42"
-		)
-		(pin "30"
-		)
-		(pin "37"
-		)
-		(pin "13"
-		)
-		(pin "9"
-		)
-		(pin "29"
-		)
-		(pin "25"
-		)
-		(pin "3"
-		)
-		(pin "39"
-		)
-		(pin "10"
-		)
-		(pin "34"
-		)
-		(pin "35"
-		)
-		(pin "11"
-		)
-		(pin "1"
-		)
-		(pin "22"
-		)
-		(pin "16"
-		)
-		(pin "56"
-		)
-		(pin "28"
-		)
-		(pin "15"
-		)
-		(pin "26"
-		)
-		(instances
-			(project "IchnaeaV1"
-				(path "/1a8ad36a-4b76-4949-97c2-661f12a0b1d9/7342cc35-6a9f-494d-986c-f265a8bd1d63/66c652f9-1522-4271-b419-016a2a2605cf"
-					(reference "U1")
-					(unit 1)
-				)
-			)
-		)
-	)
 )
