File: hw/ver1/PowerStage/IchnaeaV1.kicad_pcb (KiCad board)
At the start: 2 copper layers, 4 parts, among them U1 RP2040, U4 LTC7871

Commit message: Sync some start to the PCB design
Parts:
- added C1: 4.7uF, Capacitor_SMD:C_0603_1608Metric, F.Cu at (82.9, 71.6)
- added C10: 100nF, Capacitor_SMD:C_0603_1608Metric, F.Cu at (53.7, 30.9)
- added C11: 100nF, Capacitor_SMD:C_0603_1608Metric, F.Cu at (53.7, 33.4)
- added C12: 47pF, Capacitor_SMD:C_0603_1608Metric, F.Cu at (53.7, 35.9)
- added C13: 47pF, Capacitor_SMD:C_0603_1608Metric, F.Cu at (53.7, 38.5)
- added C14: 100nF, Capacitor_SMD:C_0603_1608Metric, F.Cu at (53.7, 41.0)
- added C15: 100nF, Capacitor_SMD:C_0603_1608Metric, F.Cu at (53.7, 43.5)
- added C16: 4.7uF, Capacitor_SMD:C_0603_1608Metric, F.Cu at (53.7, 46.0)
- added C17: Cff, Capacitor_SMD:C_0603_1608Metric_Pad1.08x0.95mm_HandSolder, F.Cu at (73.1, 55.6)
- added C18: 4.7uF, Capacitor_SMD:C_0603_1608Metric, F.Cu at (57.7, 23.4)
- added C19: 10uF, Capacitor_SMD:C_1210_3225Metric_Pad1.33x2.70mm_HandSolder, F.Cu at (90.6, 50.0)
- added C2: 100nF, Capacitor_SMD:C_0603_1608Metric, F.Cu at (82.9, 74.1)
- added C20: 10uF, Capacitor_SMD:C_1210_3225Metric_Pad1.33x2.70mm_HandSolder, F.Cu at (90.6, 54.3)
- added C21: 4.7uF, Capacitor_SMD:C_0603_1608Metric, F.Cu at (57.7, 25.9)
- added C22: 220uF, Capacitor_THT:CP_Radial_D10.0mm_P5.00mm, F.Cu at (79.3, 27.9)
- added C23: 10uF, Capacitor_SMD:C_1210_3225Metric_Pad1.33x2.70mm_HandSolder, F.Cu at (90.6, 58.5)
- added C24: 10uF, Capacitor_SMD:C_1210_3225Metric_Pad1.33x2.70mm_HandSolder, F.Cu at (90.6, 62.8)
- added C25: 220uF, Capacitor_THT:CP_Radial_D10.0mm_P5.00mm, F.Cu at (79.3, 39.5)
- added C26: 220uF, Capacitor_THT:CP_Radial_D10.0mm_P5.00mm, F.Cu at (79.3, 51.0)
- added C27: 220uF, Capacitor_THT:CP_Radial_D10.0mm_P5.00mm, F.Cu at (79.3, 62.6)
- added C28: 4.7uF, Capacitor_SMD:C_0603_1608Metric, F.Cu at (126.7, 102.6)
- added C29: 100nF, Capacitor_SMD:C_0603_1608Metric, F.Cu at (126.7, 105.1)
- added C3: 470nF, Capacitor_SMD:C_0603_1608Metric, F.Cu at (82.9, 76.6)
- added C30: 470nF, Capacitor_SMD:C_0603_1608Metric, F.Cu at (126.7, 107.6)
- added C31: 100nF, Capacitor_SMD:C_0603_1608Metric, F.Cu at (126.7, 110.1)
- added C32: 470nF, Capacitor_SMD:C_0603_1608Metric, F.Cu at (126.7, 112.6)
- added C33: 10uF, Capacitor_SMD:C_1210_3225Metric_Pad1.33x2.70mm_HandSolder, F.Cu at (131.8, 116.9)
- added C34: 4.7uF, Capacitor_SMD:C_0603_1608Metric, F.Cu at (82.9, 133.6)
- added C35: 100nF, Capacitor_SMD:C_0603_1608Metric, F.Cu at (82.9, 136.1)
- added C36: 470nF, Capacitor_SMD:C_0603_1608Metric, F.Cu at (82.9, 138.6)
- added C37: 100nF, Capacitor_SMD:C_0603_1608Metric, F.Cu at (82.9, 141.1)
- added C38: 470nF, Capacitor_SMD:C_0603_1608Metric, F.Cu at (82.9, 143.6)
- added C39: 10uF, Capacitor_SMD:C_1210_3225Metric_Pad1.33x2.70mm_HandSolder, F.Cu at (87.9, 147.8)
- added C4: 100nF, Capacitor_SMD:C_0603_1608Metric, F.Cu at (82.9, 79.1)
- added C40: 4.7uF, Capacitor_SMD:C_0603_1608Metric, F.Cu at (126.7, 133.6)
- added C41: 100nF, Capacitor_SMD:C_0603_1608Metric, F.Cu at (126.7, 136.1)
- added C42: 470nF, Capacitor_SMD:C_0603_1608Metric, F.Cu at (126.7, 138.6)
- added C43: 100nF, Capacitor_SMD:C_0603_1608Metric, F.Cu at (126.7, 141.1)
- added C44: 470nF, Capacitor_SMD:C_0603_1608Metric, F.Cu at (126.7, 143.6)
- added C45: 10uF, Capacitor_SMD:C_1210_3225Metric_Pad1.33x2.70mm_HandSolder, F.Cu at (131.8, 147.8)
- added C46: 4.7uF, Capacitor_SMD:C_0603_1608Metric, F.Cu at (126.7, 71.6)
- added C47: 100nF, Capacitor_SMD:C_0603_1608Metric, F.Cu at (126.7, 74.1)
- added C48: 470nF, Capacitor_SMD:C_0603_1608Metric, F.Cu at (126.7, 76.6)
- added C49: 100nF, Capacitor_SMD:C_0603_1608Metric, F.Cu at (126.7, 79.1)
- added C5: 470nF, Capacitor_SMD:C_0603_1608Metric, F.Cu at (82.9, 81.6)
- added C50: 470nF, Capacitor_SMD:C_0603_1608Metric, F.Cu at (126.7, 81.6)
- added C51: 10uF, Capacitor_SMD:C_1210_3225Metric_Pad1.33x2.70mm_HandSolder, F.Cu at (131.8, 85.9)
- added C52: 4.7uF, Capacitor_SMD:C_0603_1608Metric, F.Cu at (82.9, 102.6)
- added C53: 100nF, Capacitor_SMD:C_0603_1608Metric, F.Cu at (82.9, 105.1)
- added C54: 470nF, Capacitor_SMD:C_0603_1608Metric, F.Cu at (82.9, 107.6)
- added C55: 100nF, Capacitor_SMD:C_0603_1608Metric, F.Cu at (82.9, 110.1)
- added C56: 470nF, Capacitor_SMD:C_0603_1608Metric, F.Cu at (82.9, 112.6)
- added C57: 10uF, Capacitor_SMD:C_1210_3225Metric_Pad1.33x2.70mm_HandSolder, F.Cu at (87.9, 116.9)
- added C6: 10uF, Capacitor_SMD:C_1210_3225Metric_Pad1.33x2.70mm_HandSolder, F.Cu at (87.9, 85.9)
- added C7: 10uF, Capacitor_SMD:C_0603_1608Metric, F.Cu at (53.7, 23.4)
- added C8: 100nF, Capacitor_SMD:C_0603_1608Metric, F.Cu at (53.7, 25.9)
- added C9: 10uF, Capacitor_SMD:C_0603_1608Metric, F.Cu at (53.7, 28.4)
- added J1: Ext_+12v, Connector_PinSocket_2.54mm:PinSocket_1x02_P2.54mm_Vertical, F.Cu at (44.9, 57.0)
- added J2: Conn_02x12_Odd_Even, Connector_PinSocket_2.54mm:PinSocket_2x12_P2.54mm_Vertical, F.Cu at (47.4, 24.5)
- added J3: Screw_Terminal_01x01, MountingHole:MountingHole_8.4mm_M8_Pad_Via, F.Cu at (33.4, 31.3)
- added J4: Screw_Terminal_01x01, MountingHole:MountingHole_8.4mm_M8_Pad_Via, F.Cu at (33.4, 49.7)
- added J5: Screw_Terminal_01x01, MountingHole:MountingHole_8.4mm_M8_Pad_Via, F.Cu at (33.4, 68.0)
- added J6: Screw_Terminal_01x01, MountingHole:MountingHole_8.4mm_M8_Pad_Via, F.Cu at (33.4, 86.4)
- added J7: Conn_01x02_Socket, Connector_PinSocket_2.54mm:PinSocket_1x02_P2.54mm_Vertical, F.Cu at (73.3, 49.6)
- added JP1: SolderJumper_2_Bridged, Jumper:SolderJumper-2_P1.3mm_Bridged_RoundedPad1.0x1.5mm, F.Cu at (95.8, 49.7)
- added JP2: SolderJumper_2_Bridged, Jumper:SolderJumper-2_P1.3mm_Bridged_RoundedPad1.0x1.5mm, F.Cu at (95.8, 53.2)
- added L1: 4.7uH, Inductors:Bournes_L_PQ2614BLA, F.Cu at (66.3, 81.7)
- added L2: 4.7uH, Inductors:Bournes_L_PQ2614BLA, F.Cu at (110.2, 112.7)
- added L3: 4.7uH, Inductors:Bournes_L_PQ2614BLA, F.Cu at (66.3, 143.7)
- added L4: 4.7uH, Inductors:Bournes_L_PQ2614BLA, F.Cu at (110.2, 143.7)
- added L5: 4.7uH, Inductors:Bournes_L_PQ2614BLA, F.Cu at (110.2, 81.7)
- added L6: 4.7uH, Inductors:Bournes_L_PQ2614BLA, F.Cu at (66.3, 112.7)
- added Q1: MCAC80N10Y, Mosfets:TRANS_BSC076N06NS3-G, F.Cu at (89.5, 73.7)
- added Q10: MCAC80N10Y, Mosfets:TRANS_BSC076N06NS3-G, F.Cu at (89.5, 142.4)
- added Q11: MCAC80N10Y, Mosfets:TRANS_BSC076N06NS3-G, F.Cu at (133.3, 135.7)
- added Q12: MCAC80N10Y, Mosfets:TRANS_BSC076N06NS3-G, F.Cu at (133.3, 142.4)
- added Q13: MCAC80N10Y, Mosfets:TRANS_BSC076N06NS3-G, F.Cu at (133.3, 73.7)
- added Q14: MCAC80N10Y, Mosfets:TRANS_BSC076N06NS3-G, F.Cu at (133.3, 80.4)
- added Q15: MCAC80N10Y, Mosfets:TRANS_BSC076N06NS3-G, F.Cu at (89.5, 104.7)
- added Q16: MCAC80N10Y, Mosfets:TRANS_BSC076N06NS3-G, F.Cu at (89.5, 111.4)
- added Q2: MCAC80N10Y, Mosfets:TRANS_BSC076N06NS3-G, F.Cu at (89.5, 80.4)
- added Q3: BSS138, Package_TO_SOT_SMD:SOT-23, F.Cu at (68.5, 49.6)
- added Q4: BSS138, Package_TO_SOT_SMD:SOT-23, F.Cu at (68.5, 54.3)
- added Q5: BSS84, Package_TO_SOT_SMD:SOT-23, F.Cu at (68.5, 58.9)
- added Q6: BSS138, Package_TO_SOT_SMD:SOT-23, F.Cu at (68.5, 63.5)
- added Q7: MCAC80N10Y, Mosfets:TRANS_BSC076N06NS3-G, F.Cu at (133.3, 104.7)
- added Q8: MCAC80N10Y, Mosfets:TRANS_BSC076N06NS3-G, F.Cu at (133.3, 111.4)
- added Q9: MCAC80N10Y, Mosfets:TRANS_BSC076N06NS3-G, F.Cu at (89.5, 135.7)
- added R10: 1k, Resistor_SMD:R_0603_1608Metric, F.Cu at (57.7, 38.5)
- added R11: 100, Resistor_SMD:R_0603_1608Metric, F.Cu at (57.7, 41.0)
- added R12: 10k, Resistor_SMD:R_0603_1608Metric, F.Cu at (57.7, 43.5)
- added R13: 10k, Resistor_SMD:R_0603_1608Metric, F.Cu at (57.7, 46.0)
- added R14: 470k, Resistor_SMD:R_0603_1608Metric, F.Cu at (61.7, 23.4)
- added R15: 27k, Resistor_SMD:R_0603_1608Metric, F.Cu at (61.7, 25.9)
- added R16: 10k, Resistor_SMD:R_0603_1608Metric, F.Cu at (61.7, 28.4)
- added R17: 470k, Resistor_SMD:R_0603_1608Metric, F.Cu at (61.7, 30.9)
- added R18: 15k, Resistor_SMD:R_0603_1608Metric, F.Cu at (61.7, 33.4)
- added R19: 100, Resistor_SMD:R_0603_1608Metric, F.Cu at (61.7, 35.9)
- added R20: 10k, Resistor_SMD:R_0603_1608Metric, F.Cu at (61.7, 38.5)
- added R21: 10k, Resistor_SMD:R_0603_1608Metric, F.Cu at (61.7, 41.0)
- added R22: 10k, Resistor_SMD:R_0603_1608Metric, F.Cu at (61.7, 43.5)
- added R23: 10k, Resistor_SMD:R_0603_1608Metric, F.Cu at (61.7, 46.0)
- added R24: 10k, Resistor_SMD:R_0603_1608Metric, F.Cu at (65.7, 23.4)
- added R25: 10k, Resistor_SMD:R_0603_1608Metric, F.Cu at (65.7, 25.9)
- added R26: 10k, Resistor_SMD:R_0603_1608Metric, F.Cu at (65.7, 28.4)
- added R27: 68k, Resistor_SMD:R_0603_1608Metric, F.Cu at (65.7, 30.9)
- added R28: 10k, Resistor_SMD:R_0603_1608Metric, F.Cu at (65.7, 33.4)
- added R29: 10k, Resistor_SMD:R_0603_1608Metric, F.Cu at (65.7, 35.9)
- added R3: 10k, Resistor_SMD:R_0603_1608Metric, F.Cu at (82.9, 89.2)
- added R30: 10k, Resistor_SMD:R_0603_1608Metric, F.Cu at (65.7, 38.5)
- added R31: 3k, Resistor_SMD:R_0603_1608Metric, F.Cu at (65.7, 41.0)
- added R32: 1k, Resistor_SMD:R_0603_1608Metric, F.Cu at (65.7, 43.5)
- added R33: 10k, Resistor_SMD:R_0603_1608Metric, F.Cu at (65.7, 46.0)
- added R34: 100, Resistor_SMD:R_0603_1608Metric, F.Cu at (69.8, 23.4)
- added R35: 10k, Resistor_SMD:R_0603_1608Metric, F.Cu at (69.8, 25.9)
- added R36: 30k, Resistor_SMD:R_0603_1608Metric, F.Cu at (69.8, 28.4)
- added R37: 100k, Resistor_SMD:R_0603_1608Metric, F.Cu at (69.8, 30.9)
- added R38: 150k, Resistor_SMD:R_0603_1608Metric, F.Cu at (69.8, 33.4)
- added R39: 10k, Resistor_SMD:R_0603_1608Metric, F.Cu at (69.8, 35.9)
- added R4: 6.2k, Resistor_SMD:R_1206_3216Metric_Pad1.30x1.75mm_HandSolder, F.Cu at (87.9, 89.6)
- added R40: 330k, Resistor_SMD:R_0603_1608Metric, F.Cu at (69.8, 38.5)
- added R41: 787k, Resistor_SMD:R_0603_1608Metric_Pad0.98x0.95mm_HandSolder, F.Cu at (73.1, 58.2)
- added R42: 120k, Resistor_SMD:R_0603_1608Metric, F.Cu at (69.8, 41.0)
- added R43: 470k, Resistor_SMD:R_0603_1608Metric, F.Cu at (69.8, 43.5)
- added R44: 10k, Resistor_SMD:R_0603_1608Metric, F.Cu at (69.8, 46.0)
- added R45: 10k, Resistor_SMD:R_0603_1608Metric, F.Cu at (73.8, 23.4)
- added R46: 10k, Resistor_SMD:R_0603_1608Metric, F.Cu at (73.8, 25.9)
- added R47: 787k, Resistor_SMD:R_0603_1608Metric_Pad0.98x0.95mm_HandSolder, F.Cu at (73.1, 60.7)
- added R48: 10k, Resistor_SMD:R_0603_1608Metric, F.Cu at (73.8, 28.4)
- added R49: 100, Resistor_SMD:R_0603_1608Metric, F.Cu at (73.8, 30.9)
- added R5: 6.2k, Resistor_SMD:R_0603_1608Metric, F.Cu at (82.9, 91.7)
- added R50: 100, Resistor_SMD:R_0603_1608Metric, F.Cu at (73.8, 33.4)
- added R51: 10k, Resistor_SMD:R_0603_1608Metric, F.Cu at (73.8, 35.9)
- added R52: 10k, Resistor_SMD:R_0603_1608Metric, F.Cu at (73.8, 38.5)
- added R53: 10k, Resistor_SMD:R_0603_1608Metric, F.Cu at (73.8, 41.0)
- added R54: 10k, Resistor_SMD:R_0603_1608Metric, F.Cu at (73.8, 43.5)
- added R55: 0, Resistor_SMD:R_0603_1608Metric, F.Cu at (126.7, 115.1)
- added R56: 10k, Resistor_SMD:R_0603_1608Metric, F.Cu at (126.7, 117.6)
- added R57: 10k, Resistor_SMD:R_0603_1608Metric, F.Cu at (126.7, 120.2)
- added R58: 6.2k, Resistor_SMD:R_1206_3216Metric_Pad1.30x1.75mm_HandSolder, F.Cu at (131.7, 120.6)
- added R59: 6.2k, Resistor_SMD:R_0603_1608Metric, F.Cu at (126.7, 122.7)
- added R6: 10k, Resistor_SMD:R_0603_1608Metric, F.Cu at (57.7, 28.4)
- added R60: 0, Resistor_SMD:R_0603_1608Metric, F.Cu at (82.9, 146.1)
- added R61: 10k, Resistor_SMD:R_0603_1608Metric, F.Cu at (82.9, 148.6)
- added R62: 10k, Resistor_SMD:R_0603_1608Metric, F.Cu at (82.9, 151.1)
- added R63: 6.2k, Resistor_SMD:R_1206_3216Metric_Pad1.30x1.75mm_HandSolder, F.Cu at (87.9, 151.6)
- added R64: 6.2k, Resistor_SMD:R_0603_1608Metric, F.Cu at (82.9, 153.7)
- added R65: 0, Resistor_SMD:R_0603_1608Metric, F.Cu at (126.7, 146.1)
- added R66: 10k, Resistor_SMD:R_0603_1608Metric, F.Cu at (126.7, 148.6)
- added R67: 10k, Resistor_SMD:R_0603_1608Metric, F.Cu at (126.7, 151.1)
- added R68: 6.2k, Resistor_SMD:R_1206_3216Metric_Pad1.30x1.75mm_HandSolder, F.Cu at (131.7, 151.6)
- added R69: 6.2k, Resistor_SMD:R_0603_1608Metric, F.Cu at (126.7, 153.7)
- added R7: 10k, Resistor_SMD:R_0603_1608Metric, F.Cu at (57.7, 30.9)
- added R70: 0, Resistor_SMD:R_0603_1608Metric, F.Cu at (126.7, 84.1)
- added R71: 10k, Resistor_SMD:R_0603_1608Metric, F.Cu at (126.7, 86.7)
- added R72: 10k, Resistor_SMD:R_0603_1608Metric, F.Cu at (126.7, 89.2)
- added R73: 6.2k, Resistor_SMD:R_1206_3216Metric_Pad1.30x1.75mm_HandSolder, F.Cu at (131.7, 89.6)
- added R74: 6.2k, Resistor_SMD:R_0603_1608Metric, F.Cu at (126.7, 91.7)
- added R75: 0, Resistor_SMD:R_0603_1608Metric, F.Cu at (82.9, 115.1)
- added R76: 10k, Resistor_SMD:R_0603_1608Metric, F.Cu at (82.9, 117.6)
- added R77: 10k, Resistor_SMD:R_0603_1608Metric, F.Cu at (82.9, 120.2)
- added R78: 6.2k, Resistor_SMD:R_1206_3216Metric_Pad1.30x1.75mm_HandSolder, F.Cu at (87.9, 120.6)
- added R79: 6.2k, Resistor_SMD:R_0603_1608Metric, F.Cu at (82.9, 122.7)
- added R8: 10k, Resistor_SMD:R_0603_1608Metric, F.Cu at (57.7, 33.4)
- added R9: 10k, Resistor_SMD:R_0603_1608Metric, F.Cu at (57.7, 35.9)
- added SW1: SW_DIP_x03, Button_Switch_SMD:SW_DIP_SPSTx03_Slide_6.7x9.18mm_W6.73mm_P2.54mm_LowProfile_JPin, F.Cu at (92.8, 27.6)
- added TH1: 10k, Resistor_SMD:R_0402_1005Metric_Pad0.72x0.64mm_HandSolder, F.Cu at (95.2, 56.0)
- added TH2: 10k, Resistor_SMD:R_0402_1005Metric_Pad0.72x0.64mm_HandSolder, F.Cu at (95.2, 58.0)
- added U2: 74HC4051PW, Package_SO:TSSOP-14_4.4x5mm_P0.65mm, F.Cu at (92.0, 44.6)
- added U3: LTC7871, Package_QFP:LQFP-64-1EP_10x10mm_P0.5mm_EP6.5x6.5mm_ThermalVias, F.Cu at (58.9, 54.4)
- added U5: HIP2210, Package_DFN_QFN:TDFN-10-1EP_2x3mm_P0.5mm_EP0.9x2mm_ThermalVias, F.Cu at (131.1, 124.5)
- added U6: HIP2210, Package_DFN_QFN:TDFN-10-1EP_2x3mm_P0.5mm_EP0.9x2mm_ThermalVias, F.Cu at (87.3, 155.5)
- added U7: HIP2210, Package_DFN_QFN:TDFN-10-1EP_2x3mm_P0.5mm_EP0.9x2mm_ThermalVias, F.Cu at (131.1, 155.5)
- added U8: HIP2210, Package_DFN_QFN:TDFN-10-1EP_2x3mm_P0.5mm_EP0.9x2mm_ThermalVias, F.Cu at (131.1, 93.6)
- added U9: HIP2210, Package_DFN_QFN:TDFN-10-1EP_2x3mm_P0.5mm_EP0.9x2mm_ThermalVias, F.Cu at (87.3, 124.5)
- R1: value 1k -> 0
- U1: value RP2040 -> HIP2210; footprint Package_DFN_QFN:QFN-56-1EP_7x7mm_P0.4mm_EP3.2x3.2mm -> Package_DFN_QFN:TDFN-10-1EP_2x3mm_P0.5mm_EP0.9x2mm_ThermalVias
- U4: value LTC7871 -> LM1117MP-3.3; footprint Package_QFP:LQFP-64-1EP_10x10mm_P0.5mm_EP6.5x6.5mm_ThermalVias -> Package_TO_SOT_SMD:SOT-223-3_TabPin2
- moved R1 53.6 mm to (82.9, 84.1)
- moved R2 53.6 mm to (82.9, 86.7)
- moved U4 34.7 mm to (92.5, 37.2)
- moved U1 27.9 mm to (87.3, 93.6)
Connections:
- R1 pad 1: unconnected-(R1-Pad1) -> GND
- R1 pad 2: unconnected-(R1-Pad2) -> Net-(U1-RDT)
- R2 pad 1: unconnected-(R2-Pad1) -> GND
- R2 pad 2: unconnected-(R2-Pad2) -> Net-(Q2-G)
- U1 pad 1: Net-(U1-IOVDD-Pad1) -> +VSW
- U1 pad 10: Net-(U1-IOVDD-Pad1) -> Net-(Q2-G)
- U1 pad 11: unconnected-(U1-GPIO8-Pad11) -> GND
- U1 pad 2: unconnected-(U1-GPIO0-Pad2) -> Net-(U1-HB)
- U1 pad 3: unconnected-(U1-GPIO1-Pad3) -> Net-(Q1-G)
- U1 pad 4: unconnected-(U1-GPIO2-Pad4) -> Net-(Q1-S)
- U1 pad 5: unconnected-(U1-GPIO3-Pad5) -> +3.3VP
- U1 pad 6: unconnected-(U1-GPIO4-Pad6) -> Net-(U1-RDT)
- U1 pad 7: unconnected-(U1-GPIO5-Pad7) -> /PowerStage/Phase1/PWMEN
- U1 pad 8: unconnected-(U1-GPIO6-Pad8) -> /PowerStage/Phase5/PWM
- U1 pad 9: unconnected-(U1-GPIO7-Pad9) -> GND
- U4 pad 1: unconnected-(U4-SS-Pad1) -> GND
- U4 pad 2: (no net) -> +3.3VP
- U4 pad 3: unconnected-(U4-VFBLow-Pad3) -> +12P

Commit message: Mess with the buck design. Tear out previous approach.
Parts:
- added C58: 10uF, Capacitor_SMD:C_1210_3225Metric_Pad1.33x2.70mm_HandSolder, F.Cu at (76.8, 106.4)
- added C59: 10uF, Capacitor_SMD:C_1210_3225Metric_Pad1.33x2.70mm_HandSolder, F.Cu at (139.7, 78.7)
- added C60: 10uF, Capacitor_SMD:C_0603_1608Metric, F.Cu at (161.3, 21.4)
- added C61: 100nF, Capacitor_SMD:C_0603_1608Metric, F.Cu at (161.3, 23.9)
- added H1: MountingHole_Pad, MountingHole:MountingHole_3mm_Pad_Via, F.Cu at (128.6, 37.2)
- added H2: MountingHole_Pad, MountingHole:MountingHole_3mm_Pad_Via, F.Cu at (150.2, 157.8)
- added H3: MountingHole_Pad, MountingHole:MountingHole_3mm_Pad_Via, F.Cu at (74.0, 48.3)
- added H4: MountingHole_Pad, MountingHole:MountingHole_3mm_Pad_Via, F.Cu at (211.8, 121.9)
- J3, J4, J5, J6: footprint MountingHole:MountingHole_8.4mm_M8_Pad_Via -> MountingHole:MountingHole_5.3mm_M5_Pad_Via
- L1, L2, L3, L4, L5, L6: moved to B.Cu
- U1, U5, U6, U7, U8, U9: footprint Package_DFN_QFN:TDFN-10-1EP_2x3mm_P0.5mm_EP0.9x2mm_ThermalVias -> DFN:TDFN-10-1EP_4x4mm_P0.8mm_EP2.6x3mm
- U2: footprint Package_SO:TSSOP-14_4.4x5mm_P0.65mm -> Package_SO:TSSOP-16_4.4x5mm_P0.65mm
- moved J2 222.3 mm to (268.0, 52.1), turned to 180 degrees
- moved J5 189.0 mm to (222.2, 73.7)
- moved J7 186.0 mm to (259.2, 50.0)
- moved C18 180.1 mm to (237.8, 22.9)
- moved C21 180.1 mm to (237.8, 25.4)
- moved J1 180.1 mm to (225.0, 56.5)
- moved Q3 180.1 mm to (248.6, 49.1)
- moved Q4 180.1 mm to (248.6, 53.7)
- moved Q5 180.1 mm to (248.6, 58.4)
- moved Q6 180.1 mm to (248.6, 63.0)
- moved R10 180.1 mm to (237.8, 37.9)
- moved R11 180.1 mm to (237.8, 40.4)
- moved R12 180.1 mm to (237.8, 42.9)
- moved R13 180.1 mm to (237.8, 45.5)
- moved R14 180.1 mm to (241.8, 22.9)
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Connections:
- C11 pad 2: GNDD -> GND
- C12 pad 2: GNDD -> GND
- C13 pad 2: GNDD -> GND
- C14 pad 2: GNDD -> GND
- C15 pad 2: GNDD -> GND
- C31 pad 2: /PowerStage/Phase6/SNSA+ -> /PowerStage/Phase2/SNSA+
- C32 pad 2: /PowerStage/Phase6/SNSD+ -> /PowerStage/Phase2/SNSD+
- C37 pad 2: /PowerStage/Phase1/SNSA+ -> /PowerStage/Phase3/SNSA+
- C38 pad 2: /PowerStage/Phase1/SNSD+ -> /PowerStage/Phase3/SNSD+
- C4 pad 2: /PowerStage/Phase5/SNSA+ -> /PowerStage/Phase1/SNSA+
- C43 pad 2: /PowerStage/Phase2/SNSA+ -> /PowerStage/Phase4/SNSA+
- C44 pad 2: /PowerStage/Phase2/SNSD+ -> /PowerStage/Phase4/SNSD+
- C49 pad 2: /PowerStage/Phase3/SNSA+ -> /PowerStage/Phase5/SNSA+
- C5 pad 2: /PowerStage/Phase5/SNSD+ -> /PowerStage/Phase1/SNSD+
- C50 pad 2: /PowerStage/Phase3/SNSD+ -> /PowerStage/Phase5/SNSD+
- C55 pad 2: /PowerStage/Phase4/SNSA+ -> /PowerStage/Phase6/SNSA+
- C56 pad 2: /PowerStage/Phase4/SNSD+ -> /PowerStage/Phase6/SNSD+
- J2 pad 10: GNDD -> GND
- J2 pad 14: GNDD -> GND
- J2 pad 18: GNDD -> GND
- J2 pad 19: GNDD -> GND
- J2 pad 23: GNDD -> GND
- J2 pad 24: GNDD -> GND
- J2 pad 9: GNDD -> GND
- J7 pad 2: GNDD -> GND
- Q3 pad 2: GNDD -> GND
- Q4 pad 2: GNDD -> GND
- Q6 pad 2: GNDD -> GND
- R12 pad 1: GNDD -> GND
- R15 pad 1: GNDD -> GND
- R18 pad 1: GNDD -> GND
- R21 pad 1: GNDD -> GND
- R24 pad 1: GNDD -> GND
- R26 pad 1: GNDD -> GND
- R27 pad 1: GNDD -> GND
- R28 pad 1: GNDD -> GND
- R29 pad 2: GNDD -> GND
- R36 pad 1: GNDD -> GND
- R39 pad 1: GNDD -> GND
- R4 pad 2: /PowerStage/Phase5/SNSA+ -> /PowerStage/Phase1/SNSA+
- R44 pad 1: GNDD -> GND
- R45 pad 1: GNDD -> GND
- R46 pad 1: GNDD -> GND
- R48 pad 1: GNDD -> GND
- R5 pad 1: /PowerStage/Phase5/SNSD+ -> /PowerStage/Phase1/SNSD+
- R5 pad 2: /PowerStage/Phase5/SNSA+ -> /PowerStage/Phase1/SNSA+
- R51 pad 1: GNDD -> GND
- R53 pad 1: GNDD -> GND
- R58 pad 2: /PowerStage/Phase6/SNSA+ -> /PowerStage/Phase2/SNSA+
- R59 pad 1: /PowerStage/Phase6/SNSD+ -> /PowerStage/Phase2/SNSD+
- R59 pad 2: /PowerStage/Phase6/SNSA+ -> /PowerStage/Phase2/SNSA+
- R6 pad 1: GNDD -> GND
- R63 pad 2: /PowerStage/Phase1/SNSA+ -> /PowerStage/Phase3/SNSA+
- R64 pad 1: /PowerStage/Phase1/SNSD+ -> /PowerStage/Phase3/SNSD+
- R64 pad 2: /PowerStage/Phase1/SNSA+ -> /PowerStage/Phase3/SNSA+
- R68 pad 2: /PowerStage/Phase2/SNSA+ -> /PowerStage/Phase4/SNSA+
- R69 pad 1: /PowerStage/Phase2/SNSD+ -> /PowerStage/Phase4/SNSD+
- R69 pad 2: /PowerStage/Phase2/SNSA+ -> /PowerStage/Phase4/SNSA+
- R7 pad 1: GNDD -> GND
- R73 pad 2: /PowerStage/Phase3/SNSA+ -> /PowerStage/Phase5/SNSA+
- R74 pad 1: /PowerStage/Phase3/SNSD+ -> /PowerStage/Phase5/SNSD+
- R74 pad 2: /PowerStage/Phase3/SNSA+ -> /PowerStage/Phase5/SNSA+
- R78 pad 2: /PowerStage/Phase4/SNSA+ -> /PowerStage/Phase6/SNSA+
- R79 pad 1: /PowerStage/Phase4/SNSD+ -> /PowerStage/Phase6/SNSD+
- R79 pad 2: /PowerStage/Phase4/SNSA+ -> /PowerStage/Phase6/SNSA+
- R8 pad 1: GNDD -> GND
- R9 pad 1: GNDD -> GND
- TH1 pad 2: GNDD -> GND
- TH2 pad 2: GNDD -> GND
- U1 pad 8: /PowerStage/Phase5/PWM -> /PowerStage/Phase1/PWM
- U2 pad 6: GNDD -> GND
- U2 pad 7: GNDD -> GND
- U2 pad 8: GNDD -> GND
- U3 pad 12: (no net) -> unconnected-(U3-Pad12)
- U3 pad 2: (no net) -> unconnected-(U3-Pad2)
- U3 pad 26: (no net) -> unconnected-(U3-Pad26)
- U3 pad 41: (no net) -> unconnected-(U3-Pad41)
- U3 pad 43: (no net) -> unconnected-(U3-Pad43)
- U3 pad 47: (no net) -> unconnected-(U3-Pad47)
- U3 pad 55: (no net) -> unconnected-(U3-Pad55)
- U3 pad 8: (no net) -> unconnected-(U3-Pad8)
- U5 pad 8: /PowerStage/Phase6/PWM -> /PowerStage/Phase2/PWM
- U6 pad 8: /PowerStage/Phase1/PWM -> /PowerStage/Phase3/PWM
- U7 pad 8: /PowerStage/Phase2/PWM -> /PowerStage/Phase4/PWM
- U8 pad 8: /PowerStage/Phase3/PWM -> /PowerStage/Phase5/PWM
- U9 pad 8: /PowerStage/Phase4/PWM -> /PowerStage/Phase6/PWM
Other:
- board outline added: 96.5 x 96.5 mm
- copper layers 2 -> 4
- board text added: "GND"
- board text added: "VIN"
- board text added: "VOUT"

Commit message: Sync lunch work
Parts:
- C22, C25, C26, C27: moved to B.Cu
- moved J4 104.4 mm to (109.2, 139.7)
- moved J6 100.3 mm to (190.5, 139.5)
- moved C25 100.3 mm to (141.1, 90.2), turned to 0 degrees
- moved C22 96.6 mm to (141.1, 101.6)
- moved C1 83.5 mm to (42.2, 152.8)
- moved C2 83.5 mm to (42.2, 155.3)
- moved C4 83.5 mm to (42.2, 160.3)
- moved C5 83.5 mm to (42.2, 162.8)
- moved R3 83.5 mm to (64.5, 158.6)
- moved R4 83.5 mm to (49.2, 160.7)
- moved R5 83.5 mm to (42.2, 172.9)
- moved R77 83.5 mm to (64.5, 148.5)
- moved U1 83.5 mm to (64.7, 155.6)
- moved C23 83.5 mm to (60.4, 145.4)
- moved C24 83.5 mm to (60.4, 165.7)
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Routing:
- net VLOW: track 0.00 -> 153.9 mm, vias 0 -> 3
- net Net-(Q15-S): track 0.00 -> 88.5 mm, vias 0 -> 1
- net Net-(Q13-S): track 0.00 -> 52.6 mm, vias 0 -> 1
- net Net-(Q11-S): track 0.00 -> 20.9 mm, vias 0 -> 1

Commit message: Sync work to laptop
Parts:
- removed J1: Ext_+12v, Connector_PinSocket_2.54mm:PinSocket_1x02_P2.54mm_Vertical
- added C62: 220uF, Capacitor_THT:CP_Radial_D10.0mm_P5.00mm, B.Cu at (158.6, 109.2)
- added C63: 220uF, Capacitor_THT:CP_Radial_D10.0mm_P5.00mm, B.Cu at (141.0, 109.3)
- added J8: FanConnector, Connector_Molex:Molex_KK-254_AE-6410-04A_1x04_P2.54mm_Vertical, F.Cu at (127.3, 142.2)
- added R80: 10k, Resistor_SMD:R_0603_1608Metric, F.Cu at (182.4, 111.4)
- added R81: 10k, Resistor_SMD:R_0603_1608Metric, F.Cu at (180.7, 87.8)
- added R82: 10k, Resistor_SMD:R_0603_1608Metric, F.Cu at (162.0, 66.6)
- added R83: 10k, Resistor_SMD:R_0603_1608Metric, F.Cu at (137.5, 63.8)
- added R84: 10k, Resistor_SMD:R_0603_1608Metric, F.Cu at (115.4, 79.5)
- added R85: 10k, Resistor_SMD:R_0603_1608Metric, F.Cu at (119.1, 108.0)
- added R86: 10k, Resistor_SMD:R_0603_1608Metric, F.Cu at (182.4, 113.9)
- added R87: 10k, Resistor_SMD:R_0603_1608Metric, F.Cu at (177.0, 85.9)
- added R88: 10k, Resistor_SMD:R_0603_1608Metric, F.Cu at (162.0, 69.1)
- added R89: 10k, Resistor_SMD:R_0603_1608Metric, F.Cu at (136.8, 61.1)
- added R90: 10k, Resistor_SMD:R_0603_1608Metric, F.Cu at (111.5, 80.0)
- added R91: 10k, Resistor_SMD:R_0603_1608Metric, F.Cu at (117.6, 108.0)
- added R92: 10k, Resistor_SMD:R_0603_1608Metric, F.Cu at (156.4, 155.7)
- C19, C20, C23, C24, C33, C39, C45, C51, C57, C58, C59, C6: moved to B.Cu
- H1, H2, H3, H4: footprint MountingHole:MountingHole_3mm_Pad_Via -> MountingHole:MountingHole_3.2mm_M3_Pad_Via
- moved J7 156.6 mm to (131.9, 141.0)
- moved C2 140.7 mm to (178.2, 119.0)
- moved C1 140.5 mm to (178.1, 117.3)
- moved H3 138.0 mm to (181.3, 135.0)
- moved C24 132.7 mm to (162.6, 81.0), turned to 180 degrees
- moved C3 131.4 mm to (187.4, 119.1)
- moved R3 131.4 mm to (190.7, 122.2)
- moved U1 131.4 mm to (190.9, 119.1)
- moved R5 127.6 mm to (161.8, 128.5)
- moved C4 127.4 mm to (165.6, 128.4)
- moved C5 127.4 mm to (165.6, 130.9)
- moved J2 126.3 mm to (180.8, 143.5), turned to -90 degrees
- moved Q1 125.6 mm to (178.9, 122.9), turned to 0 degrees
- moved R4 116.0 mm to (161.3, 130.8)
- moved R1 104.9 mm to (178.6, 114.0)
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Connections:
- J2 pad 19: GND -> FAN_SENSE
- J2 pad 21: SYNC -> FAN_CTRL
- J2 pad 23: GND -> SYNC
- U1 pad 5: +3.3VP -> Net-(U1-VREF)
- U5 pad 5: +3.3VP -> Net-(U5-VREF)
- U6 pad 5: +3.3VP -> Net-(U6-VREF)
- U7 pad 5: +3.3VP -> Net-(U7-VREF)
- U8 pad 5: +3.3VP -> Net-(U8-VREF)
- U9 pad 5: +3.3VP -> Net-(U9-VREF)
Routing:
- net Net-(Q15-S): track 88.5 -> 14.5 mm, vias 1 -> 13
- net VLOW: track 153.9 -> 215.5 mm, vias 3 -> 6
- net Net-(Q10-D): track 0.00 -> 51.1 mm, vias 0 -> 13
- net Net-(Q7-S): track 0.00 -> 42.6 mm, vias 0 -> 13
- net Net-(Q11-S): track 20.9 -> 49.5 mm, vias 1 -> 13
- net Net-(Q16-G): track 0.00 -> 15.5 mm
- net Net-(Q1-S): track 0.00 -> 11.9 mm, vias 0 -> 13
- net Net-(U9-VREF): track 0.00 -> 8.93 mm, vias 0 -> 2
- net Net-(Q13-S): track 52.6 -> 43.6 mm, vias 1 -> 13
- net GND: track 0.00 -> 8.55 mm, vias 0 -> 17
- net Net-(Q15-G): track 0.00 -> 5.87 mm
- net +VSW: track 0.00 -> 4.91 mm
- net Net-(U9-RDT): track 0.00 -> 1.75 mm
- net Net-(U9-HB): track 0.00 -> 1.41 mm
- net /PowerStage/Phase6/PWM: track 0.00 -> 1.36 mm, vias 0 -> 1
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- added copper zone on F.Cu, net GND
- added copper zone on In2.Cu, net GND
- added copper zone on F.Cu, net Net-(Q15-S)

Commit message: Lunch effort. Add models for screw terminals. Work on power distribution planes.
Parts:
- C19, C20, C23, C24, C58, C59: moved to F.Cu
- J3, J4, J5, J6: value Screw_Terminal_01x01 -> Screw_Terminal_01x09; footprint MountingHole:MountingHole_5.3mm_M5_Pad_Via -> Connectors:CONN_74651195R_WRE
- JP1, JP2, U2, U4: moved to B.Cu
- moved C60 143.8 mm to (199.2, 160.0), turned to 90 degrees
- moved C61 142.0 mm to (201.8, 160.0), turned to 90 degrees
- moved JP1 134.1 mm to (154.3, 162.3), turned to 0 degrees
- moved JP2 131.3 mm to (154.3, 158.8), turned to 0 degrees
- moved U2 125.5 mm to (181.6, 158.8), turned to 0 degrees
- moved U4 122.4 mm to (165.1, 155.6), turned to 0 degrees
- moved TH1 111.8 mm to (208.3, 139.2), turned to 180 degrees
- moved TH2 109.4 mm to (208.3, 137.2), turned to 180 degrees
- moved C17 91.4 mm to (224.0, 141.7)
- moved C10 91.4 mm to (204.6, 117.0)
- moved C11 91.4 mm to (204.6, 119.5)
- moved C12 91.4 mm to (204.6, 122.0)
- moved C13 91.4 mm to (204.6, 124.5)
- moved C14 91.4 mm to (204.6, 127.0)
- moved C15 91.4 mm to (204.6, 129.5)
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Routing:
- net GND: track 8.55 -> 14.0 mm, vias 17 -> 10
- net Net-(Q16-G): track 15.5 -> 19.2 mm, vias 0 -> 2
- net Net-(U9-HB): track 1.41 -> 0.00 mm
- net Net-(Q15-G): track 5.87 -> 4.65 mm
- net Net-(Q15-S): track 14.5 -> 13.6 mm
- net Net-(U9-VREF): track 8.93 -> 9.68 mm
- net /PowerStage/Phase6/PWM: track 1.36 -> 0.65 mm
- net /PowerStage/Phase1/PWMEN: track 1.34 -> 0.67 mm
- net +VSW: track 4.91 -> 4.30 mm
- added copper zone on In1.Cu, net GND
- added copper zone on F.Cu, net HT
- added copper zone on In1.Cu, net HT
- added copper zone on B.Cu, net VLOW
- added copper zone on In2.Cu, net VLOW
Other:
- outline, holes or cut-outs redrawn
