File: hw/ver2/IchnaeaV2/Phase2Driver.kicad_sch (KiCad schematic)
At the start: 31 parts, among them Q6 MCAC80N10Y, Q7 MCAC80N10Y, Q8 MCAC80N10Y, Q9 MCAC80N10Y, U3 HIP2210

Commit message: Test production outputs for V2
Parts:
- R10: LCSC N/A -> C3017007
- TP19, TP20, TP21, TP22, TP23, TP49, TP50, TP51: LCSC (none) -> N/A
Changed lines of the file:
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@@
+			)
+		)
+		(property "LCSC" "N/A"
+			(at 53.34 78.74 0)
+			(effects
+				(font
+					(size 1.27 1.27)
+				)
+				(hide yes)
 			)
 		)
@@
 			)
 		)
+		(property "LCSC" "N/A"
+			(at 52.07 85.09 0)
+			(effects
+				(font
+					(size 1.27 1.27)
+				)
+				(hide yes)
+			)
+		)
 		(pin "1"
 		)
@@
 			)
 		)
+		(property "LCSC" "N/A"
+			(at 156.21 87.63 0)
+			(effects
+				(font
+					(size 1.27 1.27)
+				)
+				(hide yes)
+			)
+		)
 		(pin "1"
 		)
@@
 			)
 		)
+		(property "LCSC" "N/A"
+			(at 102.87 113.03 0)
+			(effects
+				(font
+					(size 1.27 1.27)
+				)
+				(hide yes)
+			)
+		)
 		(pin "1"
 		)
@@
 		)
 		(property "Description" "test point"
+			(at 189.23 67.31 0)
+			(effects
+				(font
+					(size 1.27 1.27)
+				)
+				(hide yes)
+			)
+		)
+		(property "LCSC" "N/A"
 			(at 189.23 67.31 0)
 			(effects
@@
 			)
 		)
+		(property "LCSC" "N/A"
+			(at 102.87 109.22 0)
+			(effects
+				(font
+					(size 1.27 1.27)
+				)
+				(hide yes)
+			)
+		)
 		(pin "1"
 		)
@@
 			)
 		)
-		(property "LCSC" "N/A"
+		(property "LCSC" "C3017007"
 			(at 163.83 87.63 0)
 			(effects
@@
 		)
 		(property "Description" "test point"
+			(at 153.67 87.63 0)
+			(effects
+				(font
+					(size 1.27 1.27)
+				)
+				(hide yes)
+			)
+		)
+		(property "LCSC" "N/A"
 			(at 153.67 87.63 0)
 			(effects
@@
 			(at 102.87 101.6 0)
 			(effects
+				(font
+					(size 1.27 1.27)
+				)
+				(hide yes)
+			)
+		)
+		(property "LCSC" "N/A"
+			(at 102.87 101.6 0)
+			(effects

Commit message: Sync schematic updates
Parts:
- R9: LCSC C21189 -> C25819
Changed lines of the file:
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@@
 			)
 		)
-		(property "LCSC" "C21189"
+		(property "LCSC" "C25819"
 			(at 71.12 107.95 0)
 			(effects
