File: hw/ver3/IchnaeaV3/PowerStage.kicad_sch (KiCad schematic)
At the start: 61 parts, among them Q1 BSS138, U2 LTC7871, U3 AP66200FVBW-13, U4 LM1117MP-5.0

Commit message: Route power control signals. Upgrade to KiCad v9.0.0.
Changed lines of the file:
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@@
 (kicad_sch
-	(version 20231120)
+	(version 20250114)
 	(generator "eeschema")
-	(generator_version "8.0")
+	(generator_version "9.0")
 	(paper "A3")
+	(text "SwitchFreq = R * 8.28kHz/kOhm\nR = 68.1k => 400kHz"
+		(exclude_from_sim no)
+		(at 102.616 269.494 0)
+		(effects
+			(font
+				(size 1.27 1.27)
+			)
+			(justify left)
+		)
+	)
+	(text "Fig.40, sets UVLO ~12v."
+		(exclude_from_sim no)
+		(at 285.75 76.2 0)
+		(effects
+			(font
+				(size 1.27 1.27)
+			)
+		)
+	)
+	(text "V5 bypass. \nPlace close to pin."
+		(exclude_from_sim no)
+		(at 127.508 81.788 0)
+		(effects
+			(font
+				(size 1.27 1.27)
+			)
+		)
+	)
+	(text "Sets max avg inductor current to ~30A. \nTrimmed with the IDAC_SETCUR register."
+		(exclude_from_sim no)
+		(at 94.234 116.84 0)
+		(effects
+			(font
+				(size 1.27 1.27)
+			)
+			(justify left)
+		)
+	)
+	(text "Corresponds to 3/4 * V5, or \n40mV peak DCR Sense. With this\nproject's inductor, that's about\n25A per phase."
+		(exclude_from_sim no)
+		(at 64.516 271.526 0)
+		(effects
+			(font
+				(size 1.27 1.27)
+			)
+			(justify left)
+		)
+	)
+	(text "10uF-25V Ceramic Caps"
+		(exclude_from_sim no)
+		(at 328.93 38.1 0)
+		(effects
+			(font
+				(size 1.27 1.27)
+			)
+		)
+	)
+	(text "Select between the current limited +VSW \noutput of the LTC7871 and the high power rail."
+		(exclude_from_sim no)
+		(at 337.566 76.2 0)
+		(effects
+			(font
+				(size 1.27 1.27)
+			)
+			(justify left)
+		)
+	)
+	(text "Voltage Feedback \nRange: 13.73V - 58.27V\nResolution: 0.3480V"
+		(exclude_from_sim no)
+		(at 30.48 270.51 0)
+		(effects
+			(font
+				(size 1.27 1.27)
+			)
+			(justify left)
+		)
+	)
+	(text "Current comparator compensation \nfrom LTSpice Sim"
+		(exclude_from_sim no)
+		(at 62.484 124.46 0)
+		(effects
+			(font
+				(size 1.27 1.27)
+			)
+		)
+	)
+	(text "Soft-Start Time Delay"
+		(exclude_from_sim no)
+		(at 154.432 117.602 0)
+		(effects
+			(font
+				(size 1.27 1.27)
+			)
+		)
+	)
+	(text "AP66300 Drop In Replacement"
+		(exclude_from_sim no)
+		(at 308.356 54.102 0)
+		(effects
+			(font
+				(size 1.27 1.27)
+			)
+		)
+	)
+	(text "Voltage References\nhttps://www.ti.com/download/kbase/volt/volt_div3.htm\n\nFBHigh: Unused\nOVHigh: 90V\nUVHigh: 15V\nOVLow: 56V"
+		(exclude_from_sim no)
+		(at 82.55 167.894 0)
+		(effects
+			(font
+				(size 1.27 1.27)
+			)
+			(justify left)
+		)
+	)
+	(text "DRVcc bypass. \nPlace close to pin."
+		(exclude_from_sim no)
+		(at 105.664 82.042 0)
+		(effects
+			(font
+				(size 1.27 1.27)
+			)
+		)
+	)
 	(junction
 		(at 62.23 116.84)
@@
 		)
 	)
-	(text "SwitchFreq = R * 8.28kHz/kOhm\nR = 68.1k => 400kHz"
-		(exclude_from_sim no)
-		(at 102.616 269.494 0)
-		(effects
-			(font
-				(size 1.27 1.27)
-			)
-			(justify left)
-		)
-	)
-	(text "Fig.40, sets UVLO ~12v."
-		(exclude_from_sim no)
-		(at 285.75 76.2 0)
-		(effects
-			(font
-				(size 1.27 1.27)
-			)
-		)
-	)
-	(text "V5 bypass. \nPlace close to pin."
-		(exclude_from_sim no)
-		(at 127.508 81.788 0)
-		(effects
-			(font
-				(size 1.27 1.27)
-			)
-		)
-	)
-	(text "Sets max avg inductor current to ~30A. \nTrimmed with the IDAC_SETCUR register."
-		(exclude_from_sim no)
-		(at 94.234 116.84 0)
-		(effects
-			(font
-				(size 1.27 1.27)
-			)
-			(justify left)
-		)
-	)
-	(text "Corresponds to 3/4 * V5, or \n40mV peak DCR Sense. With this\nproject's inductor, that's about\n25A per phase."
-		(exclude_from_sim no)
-		(at 64.516 271.526 0)
-		(effects
-			(font
-				(size 1.27 1.27)
-			)
-			(justify left)
-		)
-	)
-	(text "10uF-25V Ceramic Caps"
-		(exclude_from_sim no)
-		(at 328.93 38.1 0)
-		(effects
-			(font
-				(size 1.27 1.27)
-			)
-		)
-	)
-	(text "Select between the current limited +VSW \noutput of the LTC7871 and the high power rail."
-		(exclude_from_sim no)
-		(at 337.566 76.2 0)
-		(effects
-			(font
-				(size 1.27 1.27)
-			)
-			(justify left)
-		)
-	)
-	(text "Voltage Feedback \nRange: 13.73V - 58.27V\nResolution: 0.3480V"
-		(exclude_from_sim no)
-		(at 30.48 270.51 0)
-		(effects
-			(font
-				(size 1.27 1.27)
-			)
-			(justify left)
-		)
-	)
-	(text "Current comparator compensation \nfrom LTSpice Sim"
-		(exclude_from_sim no)
-		(at 62.484 124.46 0)
-		(effects
-			(font
-				(size 1.27 1.27)
-			)
-		)
-	)
-	(text "Soft-Start Time Delay"
-		(exclude_from_sim no)
-		(at 154.432 117.602 0)
-		(effects
-			(font
-				(size 1.27 1.27)
-			)
-		)
-	)
-	(text "AP66300 Drop In Replacement"
-		(exclude_from_sim no)
-		(at 308.356 54.102 0)
-		(effects
-			(font
-				(size 1.27 1.27)
-			)
-		)
-	)
-	(text "Voltage References\nhttps://www.ti.com/download/kbase/volt/volt_div3.htm\n\nFBHigh: Unused\nOVHigh: 90V\nUVHigh: 15V\nOVLow: 56V"
-		(exclude_from_sim no)
-		(at 82.55 167.894 0)
-		(effects
-			(font
-				(size 1.27 1.27)
-			)
-			(justify left)
-		)
-	)
-	(text "DRVcc bypass. \nPlace close to pin."
-		(exclude_from_sim no)
-		(at 105.664 82.042 0)
-		(effects
-			(font
-				(size 1.27 1.27)
-			)
-		)
-	)
 	(label "ExtVCC"
 		(at 227.33 68.58 0)
-		(fields_autoplaced yes)
 		(effects
 			(font
@@
 		(shape input)
 		(at 273.05 179.07 0)
-		(fields_autoplaced yes)
 		(effects
 			(font
@@
 		(shape input)
 		(at 182.88 154.94 180)
-		(fields_autoplaced yes)
 		(effects
 			(font
@@
 		(shape input)
 		(at 184.15 167.64 180)
-		(fields_autoplaced yes)
 		(effects
 			(font
@@
 		(shape input)
 		(at 182.88 152.4 180)
-		(fields_autoplaced yes)
 		(effects
 			(font
@@
 		(shape input)
 		(at 182.88 149.86 180)
-		(fields_autoplaced yes)
 		(effects
 			(font
@@
 		(shape output)
 		(at 184.15 172.72 180)
-		(fields_autoplaced yes)
 		(effects
 			(font
@@
 		(shape input)
 		(at 184.15 175.26 180)
-		(fields_autoplaced yes)
 		(effects
 			(font
@@
 		(shape input)
 		(at 184.15 170.18 180)
-		(fields_autoplaced yes)
 		(effects
 			(font
@@
 		(shape input)
 		(at 327.66 163.83 180)
-		(fields_autoplaced yes)
 		(effects
 			(font
@@
 			)
 		)
-		(property "Datasheet" "~"
+		(property "Datasheet" "https://www.lcsc.com/datasheet/lcsc_datasheet_2411211938_MDD-Microdiode-Semiconductor-SB10100L_C113946.pdf"
 			(at 190.5 68.58 0)
 			(effects
@@
 		(at 223.52 128.27)
 		(size 19.05 10.16)
+		(exclude_from_sim no)
+		(in_bom yes)
+		(on_board yes)
+		(dnp no)
 		(fields_autoplaced yes)
 		(stroke
@@
 		(at 223.52 102.87)
 		(size 19.05 10.16)
+		(exclude_from_sim no)
+		(in_bom yes)
+		(on_board yes)
+		(dnp no)
 		(fields_autoplaced yes)
 		(stroke
@@
 		(at 223.52 153.67)
 		(size 19.05 10.16)
+		(exclude_from_sim no)
+		(in_bom yes)
+		(on_board yes)
+		(dnp no)
 		(fields_autoplaced yes)
 		(stroke
@@
 		(at 327.66 154.94)
 		(size 21.59 12.065)
+		(exclude_from_sim no)
+		(in_bom yes)
+		(on_board yes)
+		(dnp no)
 		(fields_autoplaced yes)
 		(stroke
@@
 		(at 223.52 115.57)
 		(size 19.05 10.16)
+		(exclude_from_sim no)
+		(in_bom yes)
+		(on_board yes)
+		(dnp no)
 		(fields_autoplaced yes)
 		(stroke
@@
 		(at 223.52 140.97)
 		(size 19.05 10.16)
+		(exclude_from_sim no)
+		(in_bom yes)
+		(on_board yes)
+		(dnp no)
 		(fields_autoplaced yes)
 		(stroke
@@
 		(at 223.52 166.37)
 		(size 19.05 10.16)
+		(exclude_from_sim no)
+		(in_bom yes)
+		(on_board yes)
+		(dnp no)
 		(fields_autoplaced yes)
 		(stroke
