File: hw/ver3/IchnaeaV3/PowerStage.kicad_sch (KiCad schematic)
At the start: 61 parts, among them Q1 BSS138, U2 LTC7871, U3 AP66200FVBW-13, U4 LM1117MP-5.0

Commit message: Sync lunch work
Connections:
- net +5P: now also R22.2
- net +5V: no longer R22.2
Changed lines of the file:
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@@
 		(on_board yes)
 		(dnp no)
-		(fields_autoplaced yes)
 		(property "Reference" "#PWR040"
 			(at 182.88 163.83 0)
@@
 			)
 		)
-		(property "Value" "+5V"
-			(at 175.26 163.8299 90)
+		(property "Value" "+5P"
+			(at 172.466 162.814 90)
 			(effects
 				(font
 					(size 1.27 1.27)
 				)
-				(justify left)
+				(justify right)
 			)
 		)
