File: hw/ver3/ChargerV3/ChargerV3.kicad_pcb (KiCad board)
At the start: 4 copper layers, 100 x 100 mm, 325 parts, among them J1 Terminal Block, J10 TermEnable, J2 Terminal Block, J3 RJ45, J4 DataBusSelector, J5 FanConnector, J7 Debug, J8 SWD Debug, J9 USB_B_Micro, J902 ExtNTC, J903 ExtNTC, Q1 BSS138, Q10 HYG053N10NS1C2, Q11 HYG053N10NS1C2, Q12 BSS138, Q13 BSS138, Q14 BSS138, Q15 BSS84, Q16 BSS138, Q17 HYG053N10NS1C2, Q18 HYG053N10NS1C2, Q19 BSS138, Q2 HYG053N10NS1C2, Q20 HYG053N10NS1C2, Q21 HYG053N10NS1C2, Q22 HYG053N10NS1C2, Q23 HYG053N10NS1C2, Q24 HYG053N10NS1C2, Q25 HYG053N10NS1C2, Q26 HYG053N10NS1C2, Q27 HYG053N10NS1C2, Q29 2N7002, Q3 HYG053N10NS1C2, Q4 HYG053N10NS1C2, Q5 HYG053N10NS1C2, Q6 HYG053N10NS1C2, Q7 HYG053N10NS1C2, Q8 HYG053N10NS1C2, Q9 HYG053N10NS1C2, SW1 Boot, SW2 Reset, U1 INA180A4, U10 HIP2210, U11 HIP2210, U12 W25Q32JVZP, U13 ST1S14PHR, U16 AMS1117-5.0, U17 74HC4051PW, U18 RP2040, U19 INA180A4, U2 LTC7871, U20 TPSI3050, U21 W25Q32JVZP, U23 AMS1117-3.3, U3 AP66200FVBW-13, U5 SP3485EN, U6 HIP2210, U7 HIP2210, U8 HIP2210, U9 HIP2210, Y1 12MHz

Commit message: Sync board changes from before work started
Parts:
- removed D7: ACTIVITY, LED_SMD:LED_0805_2012Metric
- removed H1, H2: MountingHole_Pad, MountingHole:MountingHole_3.2mm_M3_Pad_Via
- removed Q19: BSS138, Package_TO_SOT_SMD:SOT-23
- removed Q29: 2N7002, Package_TO_SOT_SMD:SOT-23
- removed R107: 47k, Resistor_SMD:R_0603_1608Metric
- removed R108: 10k, Resistor_SMD:R_0603_1608Metric
- removed R109: 510, Resistor_SMD:R_0603_1608Metric
- added J6: DataOUT, Connector_RJ:RJ45_Amphenol_RJHSE538X, F.Cu at (168.8, 146.8)
- added R5: 3k, Resistor_SMD:R_0603_1608Metric, F.Cu at (178.7, 161.8)
- added R58: 3k, Resistor_SMD:R_0603_1608Metric, F.Cu at (178.7, 166.8)
- added R59: 3k, Resistor_SMD:R_0603_1608Metric, F.Cu at (178.7, 169.4)
- added R912: 3k, Resistor_SMD:R_0603_1608Metric, F.Cu at (184.7, 161.8)
- C107, C20, C22, C25, C26, L1, Q20, Q21, Q22, Q23, Q24, Q25, Q26, Q27, R75, R98: moved to B.Cu
- J3: value RJ45 -> DataIN; footprint Connector_RJ:RJ45_Amphenol_54602-x08_Horizontal -> Connector_RJ:RJ45_Amphenol_RJHSE538X
- R25: value 100 -> 3k
- moved R25 128.2 mm to (178.7, 164.3)
- moved Q23 86.9 mm to (183.7, 77.5), turned to 180 degrees
- moved Q27 80.8 mm to (183.7, 94.8), turned to 180 degrees
- moved Q25 77.9 mm to (183.7, 89.0), turned to 180 degrees
- moved R98 76.5 mm to (189.2, 110.5), turned to -90 degrees
- moved C93 76.0 mm to (189.8, 100.5)
- moved Q21 75.4 mm to (183.7, 83.2), turned to 180 degrees
- moved Q24 74.5 mm to (190.8, 94.8)
- moved R75 74.4 mm to (190.8, 110.5), turned to 90 degrees
- moved Q26 73.9 mm to (190.8, 89.0)
- moved C106 73.8 mm to (192.8, 100.5)
- moved Q22 73.3 mm to (190.8, 83.2)
- moved C107 72.4 mm to (192.2, 110.5), turned to 90 degrees
- moved Q20 68.5 mm to (190.8, 77.5)
- moved L1 62.3 mm to (204.8, 161.2)
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Connections:
- D22 pad 1: Net-(D22-K) -> LED_STATUS_0
- Q1 pad 1: Net-(Q1-G) -> CTL_LTC_PWM_EN
- R24 pad 2: Net-(Q1-G) -> CTL_LTC_PWM_EN
- R25 pad 1: Net-(Q1-G) -> Net-(J3-Pad12)
- R25 pad 2: CTL_LTC_PWM_EN -> +5V
- R67 pad 2: /ControlStage/InterConnectV1/IC_RTX_EN -> /ControlStage/InterConnectV1/IC_LED_IN_Y
- U18 pad 29: /ControlStage/InterConnectV1/IC_RTX_EN -> /ControlStage/InterConnectV1/IC_LED_IN_G
- U18 pad 30: /ControlStage/InterConnectV1/IC_ACTIVITY_LED_DRIVE -> /ControlStage/InterConnectV1/IC_LED_IN_Y
- U5 pad 2: /ControlStage/InterConnectV1/IC_RTX_EN -> /ControlStage/InterConnectV1/IC_LED_IN_Y
- U5 pad 3: /ControlStage/InterConnectV1/IC_RTX_EN -> /ControlStage/InterConnectV1/IC_LED_IN_Y
Routing:
- net CTL_LOAD_SW_EN: track 2.24 -> 28.5 mm, vias 0 -> 1
- net +12V: track 43.4 -> 18.0 mm, vias 22 -> 17
- net /PowerStage/ExtVCC: track 67.3 -> 54.9 mm, vias 8 -> 3
- net GND: track 150.2 -> 140.6 mm, vias 260 -> 251
- net +5V: track 27.0 -> 30.9 mm
- net Net-(U20-PXFR): track 2.15 -> 2.06 mm, vias 0 -> 1
Other:
- board text added: "Route 5v over here"
