File: hw/ver3/ChargerV3/PowerStage.kicad_sch (KiCad schematic)
At the start: 57 parts, among them Q1 BSS138, U2 LTC7871, U22 LM1117MP-3.3, U3 AP66200FVBW-13, U4 LM1117MP-5.0

Commit message: Nearly final charger schematic, updated with RS485 interconnect.
Parts:
- removed C11, C12, C127, C128, C129, C13, C14, C17, C19: 10uF-25V, Capacitor_SMD:C_0603_1608Metric, symbol Device:C
- removed U22: LM1117MP-3.3, Package_TO_SOT_SMD:SOT-223-3_TabPin2, symbol Regulator_Linear:LM1117MP-3.3
- removed U4: LM1117MP-5.0, Package_TO_SOT_SMD:SOT-223-3_TabPin2, symbol Regulator_Linear:LM1117MP-5.0
- added C106, C107, C93: 1uF, Capacitor_SMD:C_0603_1608Metric, symbol Device:C
- added Q20, Q21, Q22, Q23, Q24, Q25, Q26, Q27: HYG053N10NS1C2, Mosfets:TRANS_BSC076N06NS3-G, symbol ProjectMosfets:MCAC80N10Y
- added R75: 16.5k, Resistor_SMD:R_0603_1608Metric, symbol Device:R_US
- added R98: 10k, Resistor_SMD:R_0603_1608Metric, symbol Device:R_US
- added U20: TPSI3050, Package_SO:SOIC-8_7.5x5.85mm_P1.27mm, symbol GateDrivers:TPSI3050
Connections:
- net +3.3V: now also R22.2
- net +5P: no longer R22.2
- net +5V: now also C107.1, U20.3 (VDDP)
- net CTL_LOAD_SW_EN: now also R98.2, U20.1 (EN)
- net GND: now also C107.2, R75.2, R98.1, U20.4 (VSSP)
- net VLOW: now also Q20.1 (D), Q22.1 (D), Q24.1 (D), Q26.1 (D)
- net VOUT: now also Q21.1 (D), Q23.1 (D), Q25.1 (D), Q27.1 (D)
- new net: Q20.2 (G), Q21.2 (G), Q22.2 (G), Q23.2 (G), Q24.2 (G), Q25.2 (G), Q26.2 (G), Q27.2 (G), U20.8 (VDRV)
- new net: C106.2, Q20.3 (S), Q21.3 (S), Q22.3 (S), Q23.3 (S), Q24.3 (S), Q25.3 (S), Q26.3 (S), Q27.3 (S), U20.5 (VSSS)
- new net: C93.1, U20.7 (VDDH)
- new net: C106.1, C93.2, U20.6 (VDDM)
- new net: R75.1, U20.2 (PXFR)
Other:
- removed sheet PowerLoadSwitch
- note added: "6-Phase Buck Converter"
- note added: "Bootstraps high gate drive current supply from VLOW output. This is required because the LTC7871 uses an internal linear regulator to supply DRVcc and the chip will heat up excessively under higher output voltages. This provides a high efficiency/current path for both gate drive and board power."
- note added: "Gate Drive/Board Power Supply"
- note added: "Output Load Switch"
- note removed: "10uF-25V Ceramic Caps"
- moved on the sheet: C10, C15, C16, C18, C2, C20, C22, C25, C26, C3, C4, C5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

Commit message: Sync board changes from before work started
Parts:
- removed R25: 100, Resistor_SMD:R_0603_1608Metric, symbol Device:R_US
Connections:
- net CTL_LTC_PWM_EN: now also Q1.1 (G), R24.2
Changed lines of the file:
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@@
 	(text "6-Phase Buck Converter"
 		(exclude_from_sim no)
-		(at 172.212 14.478 0)
+		(at 172.72 283.464 0)
 		(effects
 			(font
@@
 	(global_label "CTL_LTC_PWM_EN"
 		(shape passive)
-		(at 133.35 148.59 0)
+		(at 125.73 148.59 0)
 		(fields_autoplaced yes)
 		(effects
@@
 		)
 		(property "Intersheetrefs" "${INTERSHEET_REFS}"
-			(at 151.3104 148.59 0)
+			(at 143.6904 148.59 0)
 			(effects
 				(font
@@
 					(unit 1)
 				)
-			)
-		)
-	)
-	(symbol
-		(lib_id "Device:R_US")
-		(at 129.54 148.59 90)
-		(mirror x)
-		(unit 1)
-		(exclude_from_sim no)
-		(in_bom yes)
-		(on_board yes)
-		(dnp no)
-		(fields_autoplaced yes)
-		(property "Reference" "R25"
-			(at 129.54 142.24 90)
-			(effects
-				(font
-					(size 1.27 1.27)
-				)
-			)
-		)
-		(property "Value" "100"
-			(at 129.54 144.78 90)
-			(effects
-				(font
-					(size 1.27 1.27)
-				)
-			)
-		)
-		(property "Footprint" "Resistor_SMD:R_0603_1608Metric"
-			(at 129.794 149.606 90)
-			(effects
-				(font
-					(size 1.27 1.27)
-				)
-				(hide yes)
-			)
-		)
-		(property "Datasheet" "~"
-			(at 129.54 148.59 0)
-			(effects
-				(font
-					(size 1.27 1.27)
-				)
-				(hide yes)
-			)
-		)
-		(property "Description" "Resistor, US symbol"
-			(at 129.54 148.59 0)
-			(effects
-				(font
-					(size 1.27 1.27)
-				)
-				(hide yes)
-			)
-		)
-		(property "Field-1" ""
-			(at 129.54 148.59 0)
-			(effects
-				(font
-					(size 1.27 1.27)
-				)
-				(hide yes)
-			)
-		)
-		(property "Digikey" "N/A"
-			(at 129.54 148.59 0)
-			(effects
-				(font
-					(size 1.27 1.27)
-				)
-				(hide yes)
-			)
-		)
-		(property "LCSC" "C22775"
-			(at 129.54 148.59 0)
-			(effects
-				(font
-					(size 1.27 1.27)
-				)
-				(hide yes)
-			)
-		)
-		(property "JLCPCB Rotation Offset" ""
-			(at 129.54 148.59 0)
-			(effects
-				(font
-					(size 1.27 1.27)
-				)
-				(hide yes)
-			)
-		)
-		(property "DigiKey" ""
-			(at 129.54 148.59 0)
-			(effects
-				(font
-					(size 1.27 1.27)
-				)
-				(hide yes)
-			)
-		)
-		(pin "1"
-		)
-		(pin "2"
-		)
-		(instances
-			(project "IchnaeaV3"
-				(path "/93408532-1ffa-463d-873c-16289d2b7987/31a930eb-86fc-490d-aa2b-31b72c4dd29d"
-					(reference "R25")
-					(unit 1)
-				)
